File: pathfinder-KiCAD/pathfinder.kicad_sch (KiCad schematic)
At the start: 13 parts, among them SW1 SW_Push, SW2 SW_Push, SW3 SW_Push, SW4 SW_Push, U1 XIAO-RP2040-DIP

Commit message: polished folder structure
Parts:
- added BZ1: Buzzer, Buzzer_Beeper:Buzzer_12x9.5RM7.6, symbol Device:Buzzer
- added R5: 100, Resistor_THT:R_Axial_DIN0204_L3.6mm_D1.6mm_P5.08mm_Horizontal, symbol Device:R
- R1, R2, R3, R4: value R -> 220
Connections:
- net GND: now also BZ1.2 (-)
- net buzzer: now reaches U1.9 (P2_D8_SCK)
- net buzzer: now also R5.2
- new net: BZ1.1 (+), R5.1
Other:
- moved on the sheet: SW1, SW2, SW3, SW4
